File: hardware/canbus-linbus-bridge/canbus-linbus-bridge.kicad_sch (KiCad schematic)
At the start: 33 parts, among them J1 USB_B_Micro, J2 UART, J3 10k NTC, J4 CANBus, J5 CANBus, J6 SWD, Q1 2N7002, Q2 2N7002, U1 MCP1754S-3302xCB, U2 STM32F042F6Px, U3 Voltage Regulator, U4 MCP2562HD

Commit message: Add linbus bridge code, board (not compiling yet)
Parts:
- removed J3: 10k NTC, TerminalBlock_TE-Connectivity:TerminalBlock_TE_282834-2_1x02_P2.54mm_Horizontal, symbol Connector:Screw_Terminal_01x02
- removed R3: 499k 1%, Resistor_SMD:R_0805_2012Metric_Pad1.20x1.40mm_HandSolder, symbol Device:R
- added C8: 1nF, Capacitor_SMD:C_0805_2012Metric_Pad1.18x1.45mm_HandSolder, symbol Device:C
- added D1: BAT42W-V, Diode_SMD:D_SOD-123, symbol Diode:BAT42W-V
- added J4: LINBus, TerminalBlock_TE-Connectivity:TerminalBlock_TE_282834-3_1x03_P2.54mm_Horizontal, symbol Connector:Screw_Terminal_01x03
- added R5, R6: 10k, Resistor_SMD:R_0805_2012Metric_Pad1.20x1.40mm_HandSolder, symbol Device:R
- added R9: 1k, Resistor_SMD:R_0805_2012Metric_Pad1.20x1.40mm_HandSolder, symbol Device:R
- added U5: TJA1021T, Package_SO:SOIC-8_3.9x4.9mm_P1.27mm, symbol Interface_CAN_LIN:TJA1021T
- JP1: renamed from JP3; footprint (none) -> Jumper:SolderJumper-2_P1.3mm_Open_TrianglePad1.0x1.5mm
- R4: value 100k 1% -> 10k
- renumbered C2 to C1, C1 to C2, C4 to C3, C3 to C4, J6 to J2, J2 to J3, J4 to J5, J5 to J6, JP1 to JP2, JP2 to JP3, R5 to R3, R6 to R8
Connections:
- net +12V: now also J4.1 (Pin_1), U5.7 (VBAT)
- net +3V3: now also R4.1, R5.1, R6.1
- net GND: now also C8.2, J4.2 (Pin_2), U5.5 (GND); no longer R4.2
- net RXD2 renamed RXD
- net RXD: now also R4.2, U5.1 (RXD)
- net SCL1: no longer names the net of U2.3 (PF1)
- net SDA1: no longer names the net of U2.2 (PF0)
- net SPI1_MISO: no longer names the net of U2.12 (PA6)
- net SPI1_MOSI: no longer names the net of U2.13 (PA7)
- net SPI1_SCK: no longer names the net of U2.11 (PA5)
- net TXD2 renamed TXD
- net TXD: now also R5.2, U5.4 (TXD)
- net VBAT_MON renamed ~{LIN_WAKE}
- net ~{LIN_WAKE}: now also R7.2, U5.3 (~{WAKE}); no longer R4.1
- net VTHERM renamed ~{LIN_SLP}
- net ~{LIN_SLP}: now also R6.2, U5.2 (~{SLP}); no longer R7.2
- net ~{SPI1_SS}: no longer names the net of U2.10 (PA4)
- new net: D1.1 (K), R9.1
- new net: D1.2 (A), U5.8 (INH)
- new net LIN: C8.1, J4.3 (Pin_3), R9.2, U5.6 (LIN)
- no-connect marks 4 -> 10
Other:
- title: CANBus Thermistor Sensor -> CANBus LINBus Bridge
- moved on the sheet: C1, C3, C5, C6, C7, F1, J1, J2, J3, J5, J6, JP1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
