File: hardware/canbus-thermistor/canbus-thermistor.kicad_sch (KiCad schematic)
At the start: 33 parts, among them J1 USB_B_Micro, J2 UART, J3 10k NTC, J4 CANBus, J5 CANBus, J6 SWD, Q1 2N7002, Q2 2N7002, U1 MCP1754S-3302xCB, U2 STM32F042F6Px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

Commit message: Add more linbus mappings, rework the bridge code
Parts:
- JP3: footprint (none) -> Jumper:SolderJumper-2_P1.3mm_Open_TrianglePad1.0x1.5mm
Changed lines of the file:
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@@
       (effects (font (size 1.27 1.27)) (justify right))
     )
-    (property "Footprint" "" (id 2) (at 232.537 119.253 0)
+    (property "Footprint" "Jumper:SolderJumper-2_P1.3mm_Open_TrianglePad1.0x1.5mm" (id 2) (at 232.537 119.253 0)
       (effects (font (size 1.27 1.27)) hide)
     )
